Commit message: Minor changes

File: gofa5/patched_GoFa5.urdf (robot description, URDF)
Before this commit: robot abb_crb15000_5_95, 10 links, 9 joints
Links:
- link base: geometry collision box size=0.0001 0.0001 0.0001
- link base_link: geometry collision mesh filename=collision/base_link.stl; visual mesh filename=visual/base_link.dae
- link flange: geometry collision box size=0.0001 0.0001 0.0001
- link link_1: geometry collision mesh filename=collision/link_1.stl; visual mesh filename=visual/link_1.dae
- link link_2: geometry collision mesh filename=collision/link_2.stl; visual mesh filename=visual/link_2.dae
- link link_3: geometry collision mesh filename=collision/link_3.stl; visual mesh filename=visual/link_3.dae
- link link_4: geometry collision mesh filename=collision/link_4.stl; visual mesh filename=visual/link_4.dae
- link link_5: geometry collision mesh filename=collision/link_5.stl; visual mesh filename=visual/link_5.dae
- link link_6: geometry collision mesh filename=collision/link_6.stl; visual mesh filename=visual/link_6.dae
- link tool0: geometry collision box size=0.0001 0.0001 0.0001
